Commit message: URDF file completed

File: master_ws/src/gator_description/src/urdf/BaseGator.URDF (robot description, URDF)
Before this commit: robot Gator, 5 links, 4 joints
Links:
- added link RightLIDAR; visual mesh filename=package://gator_description/src/urdf/RightLIDAR.stl
- added link RightTUMount; visual mesh filename=package://gator_description/src/urdf/RightTU.stl
Joints:
- added joint FrontPeg_to_RightTUMount: type fixed, parent FrontPegBoard, child RightTUMount, origin xyz=0.08255 -0.19685 0.009525 rpy=0 0 0
- added joint RightTUMount_to_RightLIDAR: type continuous, parent RightTUMount, child RightLIDAR, origin xyz=-0.04054939 -0.37181215 0.18742358 rpy=0 0 -0.78539816339

Commit message: Added GPS and IMU to URDF

File: master_ws/src/gator_description/src/urdf/BaseGator.URDF (robot description, URDF)
Before this commit: robot Gator, 7 links, 6 joints
Links:
- added link GPS; visual cylinder length=0.1 radius=0.1
- added link IMU; visual box size=0.0635 0.0635 0.0254
Joints:
- added joint Base_GPS: type fixed, parent BaseGator, child GPS, origin xyz=0.8382 0 1.97 rpy=0 0 0
- added joint Base_IMU: type fixed, parent BaseGator, child IMU, origin xyz=-0.04175 -0.483 1.1073 rpy=0 0 3.14
- joint Base_FrontPeg: origin xyz=2.14992780 0 0.892175 rpy=0 0 0 -> xyz=2.23 0 0.885 rpy=0 0 0
- joint FrontPeg_to_FrontCam: origin xyz=0.00429497 0.0139485 0.04805620 rpy=0 0 0 -> xyz=0.0065 0 0.0518 rpy=0 0 0
- joint FrontPeg_to_LeftTUMount: origin xyz=0.08255 0.19685 0.009525 rpy=0 0 0 -> xyz=0.0825 0.196 0.0128 rpy=0 0 0
- joint FrontPeg_to_RightTUMount: origin xyz=0.08255 -0.19685 0.009525 rpy=0 0 0 -> xyz=0.0825 -0.196 0.0128 rpy=0 0 0
