Commit message: Modified URDF to assume a ENU IMU

File: master_ws/src/gator_description/urdf/BaseGator.URDF (robot description, URDF)
Before this commit: robot Gator, 9 links, 8 joints
Joints:
- joint Base_IMU: origin xyz=-0.04175 -0.483 1.1073 rpy=0 0 3.14 -> xyz=-0.04175 -0.483 1.1073 rpy=3.14 0 -1.5707963

Commit message: Converter + odometer
Modified wheel odometry node to calculate linear and angular velocities to use with robot_localization.

Wrote LV -> ROS publisher of odometer.

Wrote node to convert incoming steer_angle from steering wheel angle (in degrees) to steer angle (in radians).

Added new nodes to sensors launch file

Pulled in latest copy of gator_description from master.

File: master_ws/src/gator_description/urdf/BaseGator.URDF (robot description, URDF)
Before this commit: robot Gator, 9 links, 8 joints
Joints:
- joint Base_IMU: origin xyz=-0.04175 -0.483 1.1073 rpy=3.14 0 -1.5707963 -> xyz=-0.04175 -0.483 1.1073 rpy=0 0 3.14
